File: Circuit - KiCad/PinguBot/PinguBot.kicad_sch (KiCad schematic)
At the start: 5 parts, among them U1 LM386

Commit message: Circuit Improvement
Parts:
- added BT1: Battery_Cell, symbol Device:Battery_Cell
- added C3: 0.1, symbol Device:C
- added C4, C5: C, symbol Device:C
- added D1: CQY99, LED_THT:LED_D5.0mm_IRGrey, symbol LED:CQY99
- added DisplayOled: Screw_Terminal_01x04, symbol Connector:Screw_Terminal_01x04
- added J1: Jack-DC, symbol Connector:Jack-DC
- added Microphone, MotorOne, MotorTwo, Speaker: Screw_Terminal_01x02, symbol Connector:Screw_Terminal_01x02
- added Q1: 2N2219, Package_TO_SOT_THT:TO-39-3, symbol Transistor_BJT:2N2219
- added R3, R4: R, symbol Device:R
- added ServoMotorOne, ServoMotorTwo: Screw_Terminal_01x03, symbol Connector:Screw_Terminal_01x03
- added TP1: CoaxialSwitch_Testpoint, symbol Connector:CoaxialSwitch_Testpoint
- added U2: DRV8833PW, Package_SO:TSSOP-16_4.4x5mm_P0.65mm, symbol Driver_Motor:DRV8833PW
- added U3: LM7805_TO220, Package_TO_SOT_THT:TO-220-3_Vertical, symbol Regulator_Linear:LM7805_TO220
- added U4: TSOP45xx, OptoDevice:Vishay_MOLD-3Pin, symbol Interface_Optical:TSOP45xx
- added U5: ESP32_DEVKITC, symbol EESTN5:ESP32_DEVKITC
- C1: value C_Polarized -> 220
- C2: value C_Polarized -> 10
- R1: value R -> 10
Connections:
- net at R1.1: now also C1.1, U1.5
- net at R1.2: now also C3.1
- net at C1.2: now also Speaker.1 (Pin_1)
- net at C2.1: now also U1.1 (GAIN)
- net at C2.2: now also U1.8 (GAIN)
- net GND: now reaches U1.2 (-)
- net GND: now also R2.3, U1.4 (GND), BT1.2 (-), C3.2, C4.2, C5.2, J1.2, Q1.1 (E), Speaker.2 (Pin_2), U3.2 (GND), U4.2 (GND), U5.38 (GND)
- net at U1.3 (+): now also R2.2
- net VCC-5V: now reaches U1.6 (V+)
- net VCC-5V: now also C5.1, U3.3 (VO), U4.3 (Vs), U5.19 (5V)
- net Audio_Input_TX: now reaches R2.1
- net Audio_Input_TX: now also U5.35 (TXD0)
- new net: BT1.1 (+), R3.1, TP1.C
- new net: R4.1, TP1.G
- new net: D1.1 (K), Q1.3 (C)
- new net: D1.2 (A), R3.2
- new net: Q1.2 (B), R4.2
- new net +12V: C4.1, J1.1, U3.1 (VI)
- new net Pin_Logico_5: U4.1 (OUT), U5.5 (IO34)
- no-connect marks 0 -> 2
Other:
- note added: "Audio Amplifier"
- note added: "Output Devices"
- note added: "Power Supply | Jack Connector"
- note added: "zweiter Stromkreis"
- moved on the sheet: C1, C2, R1, R2, U1

Commit message: Circuit Improvement
Parts:
- added D2: LED, symbol Device:LED
- added R5: 220, symbol Device:R
- C1: value 220 -> 220μF
- C2: value 10 -> 10μF
- C4, C5: value C -> 1μf
- R3: value R -> 100
- R4: value R -> 220
Connections:
- net GND: now also DisplayOled.4 (Pin_4), D2.1 (K)
- net 3.3V: now reaches U5.1 (3V3)
- net 3.3V: now also DisplayOled.1 (Pin_1)
- net MA2: now reaches U5.27 (IO16)
- net MA1: now reaches U5.28 (IO17)
- net STBY: now reaches U5.29 (IO5)
- net MB1: now reaches U5.30 (IO18)
- net MB2: now reaches U5.31 (IO19)
- net SDA_DISPLAY: now reaches U5.33 (IO21)
- net SDA_DISPLAY: now also DisplayOled.3 (Pin_3)
- net Microphone RX: now reaches U5.34 (RXD0)
- net SCL_DISPLAY: now reaches U5.36 (IO22)
- net SCL_DISPLAY: now also DisplayOled.2 (Pin_2)
- net +12V renamed VIN
- net Audio_Input_TX renamed Speaker TX
- net Pin_Logico_5 renamed IR_DATA
- net VCC-5V renamed 5V
- net 5V: now also R5.1
- new net: D2.2 (A), R5.2
Other:
- moved on the sheet: C1, C2, C3, C4, C5, DisplayOled, J1, Microphone, MotorOne, MotorTwo, R1, R2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
